File: boards/v1/caps-lock-buzzer.sch (EAGLE design)
At the start: 10 parts, among them Q1 FMMT619TA, U1 PIC16F1459-I/SS

Commit message: Cleaned up for video
Other:
- note added: "35 mA"
- note added: "Buzzer and Transistor Switch"
- note added: "Decoupling"
- note added: "PIC16F1459 and USB"
- note added: "Programmer"
- note removed: "Lower cost and more readily available substitute for 0.1µF 50V caps is Kemet #C1206C104K5RAC7867"
- moved on the sheet: C1, C2, C3, D1, J1, LS1, Q1, R1, U1
