File: boards/v2/caps-lock-buzzer.brd (EAGLE design)
At the start: 25.4 x 25.4 mm, 14 parts, among them Q1 FMMT619TA, SW1 KMR211NGLFS, U1 PIC16F1459-I/SS, U2 PRTR5V0U2X

Commit message: Fixed LED resistor value.
Parts:
- R2: value 2.2k -> 1k
Changed lines of the file:
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@@
 <attribute name="VENDOR" value="NXP" x="8.255" y="17.62125" size="1.778" layer="27" rot="R180" display="off"/>
 </element>
-<element name="R2" library="rcl" package="R0805" value="2.2k" x="22.86" y="16.51" smashed="yes" rot="MR270"/>
+<element name="R2" library="rcl" package="R0805" value="1k" x="22.86" y="16.51" smashed="yes" rot="MR270"/>
 <element name="USER1" library="microbuilder" package="CHIPLED_0805_NOOUTLINE" value="RED" x="22.86" y="16.51" smashed="yes" rot="R180"/>
 <element name="SW1" library="adafruit" package="KMR2" value="KMR211NGLFS " x="2.54" y="8.89" smashed="yes" rot="R270"/>
