File: boards/v2/caps-lock-buzzer.sch (EAGLE design)
At the start: 14 parts, among them Q1 FMMT619TA, SW1 KMR211NGLFS, U1 PIC16F1459-I/SS, U2 PRTR5V0U2X

Commit message: Fixed LED resistor value.
Parts:
- R2: value 2.2k -> 1k
Changed lines of the file:
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@@
 <part name="SUPPLY2" library="supply2" deviceset="GND" device=""/>
 <part name="P+3" library="supply1" deviceset="+5V" device=""/>
-<part name="R2" library="rcl" deviceset="R-US_" device="R0805" value="2.2k"/>
+<part name="R2" library="rcl" deviceset="R-US_" device="R0805" value="1k"/>
 <part name="USER1" library="microbuilder" deviceset="LED" device="0805_NOOUTLINE" value="RED"/>
 <part name="P+5" library="supply1" deviceset="+5V" device=""/>
